File: Esquematico V4/_autosave-amiplanta.kicad_pcb (KiCad board)
At the start: 2 copper layers, 50 parts, among them J1 Jack-DC, J2 USB_B_Micro, Q1 SS8050-G, Q2 SS8050-G, U2 MAX98357AETE+, U3 ESP32-WROOM-32, U7 CP2102N-Axx-xQFN28

Commit message: Desarrollo PCB
Parts:
- moved Camp1 125.0 mm to (35.0, 48.2)
- moved Camp2 125.0 mm to (35.0, 52.2)
- moved U2 124.9 mm to (41.0, 51.0)
- moved CReg1 124.9 mm to (53.5, 45.1)
- moved CReg2 124.9 mm to (53.5, 41.4)
- moved Cbl1 124.9 mm to (55.0, 58.5)
- moved Cbl2 124.9 mm to (54.8, 62.2)
- moved DUSB1 124.9 mm to (60.2, 61.2)
- moved DUl1 124.9 mm to (60.2, 58.5)
- moved DUl2 124.9 mm to (60.2, 56.5)
- moved DUl3 124.9 mm to (60.2, 54.2)
- moved Q1 124.9 mm to (44.8, 51.8)
- moved Q2 124.9 mm to (52.2, 51.6)
- moved RDTR1 124.9 mm to (48.5, 50.5)
- moved RRTS1 124.9 mm to (48.5, 52.8)
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