File: Esquematico V4/Componentes/amiplanta.kicad_pcb (KiCad board)
At the start: 2 copper layers, 50 parts, among them J1 Jack-DC, J2 USB_B_Micro, Q1 SS8050-G, Q2 SS8050-G, U2 MAX98357AETE+, U3 ESP32-WROOM-32, U7 CP2102N-Axx-xQFN28

Commit message: Desarrollo PCB
Parts:
- moved R_rstbl1 132.4 mm to (47.1, 68.3), turned to 90 degrees
- moved Ractbl1 129.4 mm to (43.9, 68.3)
- moved RRXD0 127.7 mm to (58.1, 52.3)
- moved RTXD0 127.7 mm to (56.1, 52.3)
- moved DUl2 126.9 mm to (58.1, 59.6)
- moved DUl3 126.9 mm to (58.1, 61.6)
- moved DUSB1 126.9 mm to (58.1, 66.3)
- moved DUl1 126.9 mm to (58.1, 63.6)
- moved Cbl1 126.4 mm to (53.4, 60.6), turned to 0 degrees
- moved U2 126.4 mm to (39.4, 54.9), turned to 90 degrees
- moved Camp2 126.3 mm to (33.6, 53.6)
- moved Camp1 126.2 mm to (33.6, 51.6)
- moved CReg1 126.2 mm to (52.1, 46.8)
- moved CReg2 126.2 mm to (52.1, 43.1)
- moved Cbl2 126.2 mm to (53.4, 64.0)
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Routing:
- net GNDREF: track 0.00 -> 75.4 mm
- net GND: track 0.00 -> 70.0 mm
- net +3V3: track 0.00 -> 68.3 mm
- net /ESP32/SCL: track 0.00 -> 61.4 mm
- net /ESP32/SDA: track 0.00 -> 54.9 mm
- net +5V_Jack: track 0.00 -> 36.1 mm
- net BOOT: track 0.00 -> 34.8 mm, vias 0 -> 1
- net /Sensores/Amp-: track 0.00 -> 27.7 mm
- net +5V: track 0.00 -> 26.0 mm
- net /CP2102N-A02-GQFN28(Bootloader)/DTR: track 0.00 -> 24.9 mm
- net /Sensores/dt: track 0.00 -> 23.9 mm
- net EN: track 0.00 -> 22.6 mm
- net /Sensores/Amp+: track 0.00 -> 22.4 mm
- net /Sensores/dh: track 0.00 -> 20.3 mm
- net Net-(Din1-Pad2): track 0.00 -> 18.0 mm
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