File: EsquematicoV4/pantallaOled.kicad_sch (KiCad schematic)
At the start: 1 part

Commit message: Correciones Finales Esquemático - Revisar error con huella del Amplificador de Sonido
Parts:
- Joled1: footprint Connector_JST:JST_EH_B4B-EH-A_1x04_P2.50mm_Vertical -> Connector_Molex:Molex_KK-396_5273-04A_1x04_P3.96mm_Vertical
Changed lines of the file:
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@@
     (property "Reference" "Joled1" (id 0) (at 146.685 83.82 0))
     (property "Value" "Conn_01x04_Female" (id 1) (at 146.685 86.36 0))
-    (property "Footprint" "Connector_JST:JST_EH_B4B-EH-A_1x04_P2.50mm_Vertical" (id 2) (at 146.05 91.44 0)
+    (property "Footprint" "Connector_Molex:Molex_KK-396_5273-04A_1x04_P3.96mm_Vertical" (id 2) (at 146.05 91.44 0)
       (effects (font (size 1.27 1.27)) hide)
     )
